File: Hardware/3b-equalizer.kicad_sch (KiCad schematic)
At the start: 45 parts, among them U1 TL074, U2 TL074

Commit message: Calculated input impedance of buffer amp stage
Signed-off-by: bebenlebricolo <benoittarrade@hotmail.fr>
Parts:
- removed U1, U2: TL074, symbol Amplifier_Operational:TL074
- added U1, U3: MC33079, symbol Amplifier_Operational:MC33079
Connections:
- net +15V: now also U1.4 (V+)
- net -15V: now also U1.11 (V-)
- net EqOutput: now also U3.7
- net GNDA: now also U3.5 (+)
- net at C5.2, R10.1: now also U1.12 (+)
- net at C9.2, R16.1, R18.2: now also U1.1
- net at C10.1, R14.1, R17.1: now also U1.14
- net at R15.1, R17.2: now also U1.13 (-)
- net at C8.2, R25.1, R26.2: now also U1.7
- net at C7.1, R13.1: now also U1.5 (+)
- net at C6.1, R9.1: now also U1.3 (+)
- net at R11.1, R16.2: now also U1.2 (-)
- net at R20.1, R21.1, R22.1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: now also U3.6 (-)
- net at R24.1, R25.2: now also U1.6 (-)
- net at C14.2, R27.1: now also U1.10 (+)
- net at C15.1, R28.1, R30.1: now also U1.8
- net at R29.1, R30.2: now also U1.9 (-)
